File: exemplo_curso.sch (KiCad schematic (older format))
At the start: 5 parts

Commit message: Cap unit added
Parts:
- C?: value 20n -> 20nF
Changed lines of the file:
@@
 EESchema Schematic File Version 4
+LIBS:exemplo_curso-cache
 EELAYER 30 0
 EELAYER END
@@
 P 3450 3700
 F 0 "C?" V 3135 3700 50  0000 C CNN
-F 1 "20n" V 3226 3700 50  0000 C CNN
+F 1 "20nF" V 3226 3700 50  0000 C CNN
 F 2 "" H 3450 3700 50  0001 C CNN
 F 3 "~" H 3450 3700 50  0001 C CNN

Commit message: Added footprints
Parts:
- C1: renamed from C?; footprint (none) -> Capacitor_THT:C_Disc_D3.0mm_W1.6mm_P2.50mm
- R1, R2, R3: renamed from R?; footprint (none) -> Resistor_THT:R_Axial_DIN0207_L6.3mm_D2.5mm_P10.16mm_Horizontal
- gave numbers to parts that had none: 1
Other:
- moved on the sheet: C1, Q1, R1, R2, R3
Changed lines of the file:
@@
 $EndDescr
 $Comp
-L pspice:R R?
+L pspice:R R1
 U 1 1 5D93A3C7
-P 3950 3700
-F 0 "R?" V 3745 3700 50  0000 C CNN
-F 1 "1k" V 3836 3700 50  0000 C CNN
-F 2 "" H 3950 3700 50  0001 C CNN
-F 3 "~" H 3950 3700 50  0001 C CNN
-	1    3950 3700
+P 4250 3600
+F 0 "R1" V 4045 3600 50  0000 C CNN
+F 1 "1k" V 4136 3600 50  0000 C CNN
+F 2 "Resistor_THT:R_Axial_DIN0207_L6.3mm_D2.5mm_P10.16mm_Horizontal" H 4250 3600 50  0001 C CNN
+F 3 "~" H 4250 3600 50  0001 C CNN
+	1    4250 3600
 	0    1    1    0
 $EndComp
 $Comp
-L pspice:R R?
+L pspice:R R3
 U 1 1 5D93B60F
-P 5200 4150
-F 0 "R?" H 5132 4104 50  0000 R CNN
-F 1 "10k" H 5132 4195 50  0000 R CNN
-F 2 "" H 5200 4150 50  0001 C CNN
-F 3 "~" H 5200 4150 50  0001 C CNN
-	1    5200 4150
+P 5500 4050
+F 0 "R3" H 5432 4004 50  0000 R CNN
+F 1 "10k" H 5432 4095 50  0000 R CNN
+F 2 "Resistor_THT:R_Axial_DIN0207_L6.3mm_D2.5mm_P10.16mm_Horizontal" H 5500 4050 50  0001 C CNN
+F 3 "~" H 5500 4050 50  0001 C CNN
+	1    5500 4050
 	-1   0    0    1
 $EndComp
 $Comp
-L power:GND #PWR?
+L power:GND #PWR01
 U 1 1 5D93D66F
-P 4600 4500
-F 0 "#PWR?" H 4600 4250 50  0001 C CNN
-F 1 "GND" H 4605 4327 50  0000 C CNN
-F 2 "" H 4600 4500 50  0001 C CNN
-F 3 "" H 4600 4500 50  0001 C CNN
-	1    4600 4500
+P 4900 4400
+F 0 "#PWR01" H 4900 4150 50  0001 C CNN
+F 1 "GND" H 4905 4227 50  0000 C CNN
+F 2 "" H 4900 4400 50  0001 C CNN
+F 3 "" H 4900 4400 50  0001 C CNN
+	1    4900 4400
 	1    0    0    -1
 $EndComp
 Wire Wire Line
-	4600 4500 4600 4400
+	4900 4400 4900 4300
 Wire Wire Line
-	4600 3700 4200 3700
+	4900 3600 4500 3600
 Wire Wire Line
-	5200 4400 4600 4400
-Connection ~ 4600 4400
+	5500 4300 4900 4300
+Connection ~ 4900 4300
 Wire Wire Line
-	4600 3700 4900 3700
-Connection ~ 4600 3700
+	4900 3600 5200 3600
+Connection ~ 4900 3600
 Wire Wire Line
-	4600 4400 4600 4200
+	4900 4300 4900 4100
 $Comp
-L pspice:R R?
+L pspice:R R2
 U 1 1 5D93D300
-P 4600 3950
-F 0 "R?" H 4668 3996 50  0000 L CNN
-F 1 "510k" H 4668 3905 50  0000 L CNN
-F 2 "" H 4600 3950 50  0001 C CNN
-F 3 "~" H 4600 3950 50  0001 C CNN
-	1    4600 3950
+P 4900 3850
+F 0 "R2" H 4968 3896 50  0000 L CNN
+F 1 "510k" H 4968 3805 50  0000 L CNN
+F 2 "Resistor_THT:R_Axial_DIN0207_L6.3mm_D2.5mm_P10.16mm_Horizontal" H 4900 3850 50  0001 C CNN
+F 3 "~" H 4900 3850 50  0001 C CNN
+	1    4900 3850
 	1    0    0    -1
 $EndComp
 $Comp
-L Transistor_BJT:2SC1815 Q?
+L Transistor_BJT:2SC1815 Q1
 U 1 1 5D93F8B8
-P 5100 3700
-F 0 "Q?" H 5290 3746 50  0000 L CNN
-F 1 "2SC1815" H 5290 3655 50  0000 L CNN
-F 2 "Package_TO_SOT_THT:TO-92_Inline" H 5300 3625 50  0001 L CIN
-F 3 "https://media.digikey.com/pdf/Data%20Sheets/Toshiba%20PDFs/2SC1815.pdf" H 5100 3700 50  0001 L CNN
-	1    5100 3700
+P 5400 3600
+F 0 "Q1" H 5590 3646 50  0000 L CNN
+F 1 "2SC1815" H 5590 3555 50  0000 L CNN
+F 2 "Package_TO_SOT_THT:TO-92_Inline" H 5600 3525 50  0001 L CIN
+F 3 "https://media.digikey.com/pdf/Data%20Sheets/Toshiba%20PDFs/2SC1815.pdf" H 5400 3600 50  0001 L CNN
+	1    5400 3600
 	1    0    0    -1
 $EndComp
 $Comp
-L pspice:C C?
+L pspice:C C1
 U 1 1 5D93FC17
-P 3450 3700
-F 0 "C?" V 3135 3700 50  0000 C CNN
-F 1 "20nF" V 3226 3700 50  0000 C CNN
-F 2 "" H 3450 3700 50  0001 C CNN
-F 3 "~" H 3450 3700 50  0001 C CNN
-	1    3450 3700
+P 3750 3600
+F 0 "C1" V 3435 3600 50  0000 C CNN
+F 1 "20nF" V 3526 3600 50  0000 C CNN
+F 2 "Capacitor_THT:C_Disc_D3.0mm_W1.6mm_P2.50mm" H 3750 3600 50  0001 C CNN
+F 3 "~" H 3750 3600 50  0001 C CNN
+	1    3750 3600
 	0    1    1    0
 $EndComp
